Commit message: changed name of all base_links to argo_base. Still have to change in the nav_stack.Odom message doesnot have issues now.

File: src/argo_description/urdf/argo_urdf_2.xacro (robot description, xacro)
@@ -437,5 +437,5 @@
       <sick_lms1xx_mount prefix="base" topic="scan"/>
       <joint name="laser_mount_joint" type="fixed">
-        <origin xyz="$(optenv ARGO_LMS1XX_XYZ 0.2206 0.0 0.00635)"
+        <origin xyz="$(optenv ARGO_LMS1XX_XYZ 0.2206 0.0 0.0835)"
                 rpy="$(optenv ARGO_LMS1XX_RPY 0.0 0.0 0.0)" />
         <parent link="argo_base" />
@@ -457,6 +457,6 @@
     <link name="imu_link"/>
     <joint name="imu_joint" type="fixed">
-      <origin xyz="$(optenv ARGO_IMU_XYZ 0.19 0 0.149)" rpy="$(optenv ARGO_IMU_RPY 0 -1.5708 3.1416)" />
-      <parent link="base_link" />
+      <origin xyz="$(optenv ARGO_IMU_XYZ -0.0287146112802265 2.27427526650059E-06 -0.0381581636610044)" rpy="$(optenv ARGO_IMU_RPY 0 -1.5708 3.1416)" />
+      <parent link="argo_base" />
       <child link="imu_link" />
     </joint>

Commit message: All Working. Map Generating. Decorations to the argo to be done. Will create a different branch for that. Also, there is mismatch in laser upadate rate. Modification needs to be done there as well.

File: src/argo_description/urdf/argo_urdf_2.xacro (robot description, xacro)
@@ -11,5 +11,5 @@
   <xacro:include filename="$(find argo_description)/urdf/accessories/sensor_arch.urdf.xacro"/>
     <property name="M_PI" value="3.14159"/>
-<link name="base_link"/>
+<!--<link name="base_link"/>-->
   <link
     name="argo_base">
@@ -52,9 +52,9 @@
     </collision>
   </link>
-  <joint name="base_link_joint" type="fixed">
+ <!-- <joint name="base_link_joint" type="fixed">
       <origin xyz="0 0 0" rpy="0 0 0" />
       <parent link="base_link" />
       <child link="argo_base" />
-    </joint>
+    </joint>-->
   <link
     name="FLW">
@@ -437,5 +437,5 @@
       <sick_lms1xx_mount prefix="base" topic="scan"/>
       <joint name="laser_mount_joint" type="fixed">
-        <origin xyz="$(optenv ARGO_LMS1XX_XYZ 0.2206 0.0 0.0835)"
+        <origin xyz="$(optenv ARGO_LMS1XX_XYZ 0.2206 0.0 0.135)"
                 rpy="$(optenv ARGO_LMS1XX_RPY 0.0 0.0 0.0)" />
         <parent link="argo_base" />

Commit message: added willow garage world

File: src/argo_description/urdf/argo_urdf_2.xacro (robot description, xacro)
@@ -13,5 +13,5 @@
 <!--<link name="base_link"/>-->
   <link
-    name="argo_base">
+    name="base_link">
     <inertial>
       <origin
@@ -55,5 +55,5 @@
       <origin xyz="0 0 0" rpy="0 0 0" />
       <parent link="base_link" />
-      <child link="argo_base" />
+      <child link="base_link" />
     </joint>-->
   <link
@@ -105,5 +105,5 @@
       rpy="0 -1.1994E-16 0" />
     <parent
-      link="argo_base" />
+      link="base_link" />
     <child
       link="FLW" />
@@ -159,5 +159,5 @@
       rpy="0 -1.1994E-16 0" />
     <parent
-      link="argo_base" />
+      link="base_link" />
     <child
       link="MLW" />
@@ -213,5 +213,5 @@
       rpy="0 -1.1994E-16 0" />
     <parent
-      link="argo_base" />
+      link="base_link" />
     <child
       link="RLW" />
@@ -267,5 +267,5 @@
       rpy="0 0 0" />
     <parent
-      link="argo_base" />
+      link="base_link" />
     <child
       link="FRW" />
@@ -321,5 +321,5 @@
       rpy="0 -1.1994E-16 0" />
     <parent
-      link="argo_base" />
+      link="base_link" />
     <child
       link="MRW" />
@@ -375,5 +375,5 @@
       rpy="0 -0.010714 0" />
     <parent
-      link="argo_base" />
+      link="base_link" />
     <child
       link="RRW" />
@@ -439,14 +439,14 @@
         <origin xyz="$(optenv ARGO_LMS1XX_XYZ 0.2206 0.0 0.135)"
                 rpy="$(optenv ARGO_LMS1XX_RPY 0.0 0.0 0.0)" />
-        <parent link="argo_base" />
+        <parent link="base_link" />
         <child link="base_laser_mount" />
       </joint>
   <!--  <xacro:if value="$(arg kinect_enabled)">
-      <xacro:sensor_arch prefix="" parent="argo_base">
+      <xacro:sensor_arch prefix="" parent="base_link">
         <origin xyz="-0.35 0 0.51" rpy="0 0 -3.14"/>
       </xacro:sensor_arch>
       <joint name="kinect_frame_joint" type="fixed">
         <origin xyz="$(optenv ARGO_KINECT_XYZ 0 0 0)" rpy="$(optenv ARGO_KINECT_RPY 0 0.18 3.14)" />
-        <parent link="argo_base"/>
+        <parent link="base_link"/>
         <child link="camera_link"/>
       </joint>
@@ -458,5 +458,5 @@
     <joint name="imu_joint" type="fixed">
       <origin xyz="$(optenv ARGO_IMU_XYZ -0.0287146112802265 2.27427526650059E-06 -0.0381581636610044)" rpy="$(optenv ARGO_IMU_RPY 0 -1.5708 3.1416)" />
-      <parent link="argo_base" />
+      <parent link="base_link" />
       <child link="imu_link" />
     </joint>
